File: Bubbler/Bubbler.sch (EAGLE design)
At the start: 72 parts, among them SW1 SWITCH-DIP-GDH-02, SW2 ITT-SWITCH-KSS-G, U1 STM32F41X-100P, U2 SPANSION-S25FL256, U3 LM4890, U4 BIPOLAR-PMBT6428, U5 USBLC6-2, U6 TLV1117, U7 MOLEX-1.25-WTB-RA-CONN-2POS, X2 CM415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

Commit message: Corrected expansion connectors
Connections:
- new net CARD0_ID: CARD0.P22, U1.PC2/SPI2_MISO/ADC123_IN12
- new net CARD1_ID: CARD1.P22, U1.PE0/FSMC_NBL0/DCMI_D2
- net EXT0_11: no longer U1.PE9/FSMC_D6/TIM1_CH1
- net EXT1_11: no longer U1.PE11/FSMC_D8/TIM_CH2
- net EXT1_12: no longer U1.PE0/FSMC_NBL0/DCMI_D2, U1.PE10/FSMC_D7
- net GND: no longer CARD0.P22, CARD1.P22
Changed lines of the file:
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@@
-</segment>
-</net>
-<net name="EXT0_11" class="0">
-<segment>
-<pinref part="U1" gate="G$1" pin="PE9/FSMC_D6/TIM1_CH1"/>
-<wire x1="182.88" y1="33.02" x2="185.42" y2="33.02" width="0.1524" layer="91"/>
-<label x="185.42" y="33.02" size="1.778" layer="95"/>
-</segment>
-</net>
-<net name="EXT1_11" class="0">
-<segment>
-<pinref part="U1" gate="G$1" pin="PE11/FSMC_D8/TIM_CH2"/>
-<wire x1="182.88" y1="27.94" x2="185.42" y2="27.94" width="0.1524" layer="91"/>
-<label x="185.42" y="27.94" size="1.778" layer="95"/>
 </segment>
 </net>
@@
 </segment>
 </net>
-<net name="EXT1_12" class="0">
+<net name="CARD1_ID" class="0">
 <segment>
 <pinref part="U1" gate="G$1" pin="PE0/FSMC_NBL0/DCMI_D2"/>
@@
 <label x="185.42" y="55.88" size="1.778" layer="95"/>
 </segment>
-<segment>
-<pinref part="U1" gate="G$1" pin="PE10/FSMC_D7"/>
-<wire x1="182.88" y1="30.48" x2="185.42" y2="30.48" width="0.1524" layer="91"/>
-<label x="185.42" y="30.48" size="1.778" layer="95"/>
+</net>
+<net name="CARD0_ID" class="0">
+<segment>
+<pinref part="U1" gate="G$1" pin="PC2/SPI2_MISO/ADC123_IN12"/>
+<wire x1="182.88" y1="132.08" x2="185.42" y2="132.08" width="0.1524" layer="91"/>
+<label x="185.42" y="132.08" size="1.778" layer="95"/>
 </segment>
 </net>
@@
 <wire x1="124.46" y1="0" x2="124.46" y2="5.08" width="0.1524" layer="91"/>
 <wire x1="124.46" y1="5.08" x2="124.46" y2="10.16" width="0.1524" layer="91"/>
-<wire x1="124.46" y1="10.16" x2="124.46" y2="20.32" width="0.1524" layer="91"/>
-<wire x1="124.46" y1="20.32" x2="124.46" y2="63.5" width="0.1524" layer="91"/>
+<wire x1="124.46" y1="10.16" x2="124.46" y2="63.5" width="0.1524" layer="91"/>
 <wire x1="124.46" y1="63.5" x2="99.06" y2="63.5" width="0.1524" layer="91"/>
 <wire x1="99.06" y1="0" x2="124.46" y2="0" width="0.1524" layer="91"/>
@@
 <pinref part="CARD0" gate="G$1" pin="P28"/>
 <pinref part="CARD0" gate="G$1" pin="P30"/>
-<pinref part="CARD0" gate="G$1" pin="P22"/>
-<wire x1="99.06" y1="20.32" x2="124.46" y2="20.32" width="0.1524" layer="91"/>
-<junction x="124.46" y="20.32"/>
 </segment>
 <segment>
@@
 <wire x1="205.74" y1="0" x2="205.74" y2="5.08" width="0.1524" layer="91"/>
 <wire x1="205.74" y1="5.08" x2="205.74" y2="10.16" width="0.1524" layer="91"/>
-<wire x1="205.74" y1="10.16" x2="205.74" y2="20.32" width="0.1524" layer="91"/>
-<wire x1="205.74" y1="20.32" x2="205.74" y2="63.5" width="0.1524" layer="91"/>
+<wire x1="205.74" y1="10.16" x2="205.74" y2="63.5" width="0.1524" layer="91"/>
 <wire x1="205.74" y1="63.5" x2="180.34" y2="63.5" width="0.1524" layer="91"/>
 <wire x1="180.34" y1="0" x2="205.74" y2="0" width="0.1524" layer="91"/>
@@
 <pinref part="CARD1" gate="G$1" pin="P26"/>
 <pinref part="CARD1" gate="G$1" pin="P5"/>
-<pinref part="CARD1" gate="G$1" pin="P22"/>
-<wire x1="180.34" y1="20.32" x2="205.74" y2="20.32" width="0.1524" layer="91"/>
-<junction x="205.74" y="20.32"/>
 </segment>
 <segment>
@@
 </segment>
 </net>
+<net name="CARD0_ID" class="0">
+<segment>
+<pinref part="CARD0" gate="G$1" pin="P22"/>
+<wire x1="99.06" y1="20.32" x2="101.6" y2="20.32" width="0.1524" layer="91"/>
+<label x="101.6" y="20.32" size="1.778" layer="95"/>
+</segment>
+</net>
+<net name="CARD1_ID" class="0">
+<segment>
+<pinref part="CARD1" gate="G$1" pin="P22"/>
+<wire x1="180.34" y1="20.32" x2="182.88" y2="20.32" width="0.1524" layer="91"/>
+<label x="182.88" y="20.32" size="1.778" layer="95"/>
+</segment>
+</net>
