File: dev/Lepton/Lepton.sch (EAGLE design)
At the start: 64 parts, among them J1 M12, J2 M12, Q2 CM415, U1 CC3000, U2 STM32F100R4T6B, U3 STM32-JTAG-FFC, U4 SILICONLABS-HUMIDITY-SI7005, U5 FREESCALE-PRESSURE-MPL3115A2, U6 MMA8653FC, X1 USBPCB

Commit message: Updated board with smaller components, micro USB, and mounting holes
Parts:
- removed Q1: (no value), Pygmy:CRYSTAL5X3
- removed Q2: CM415, Pygmy:CM415
- added JP1: USB-MICROB, SparkFun-Connectors:USB-MICROB
- added X2: CRYSTAL-KYOCERA-ST3215SB, Pygmy:CRYSTAL-KYOCERA-ST3215SB
- C1, C12, C13, C14, C15, C16, C17, C18, C2, C3, C4, C5, C6, C7, C8, C9: device rcl:C-USC0402 -> rcl:C-USC0201
- C10, C11: device rcl:C-USC0805 -> rcl:C-USC0603
- R1, R10, R11, R12, R13, R14, R15, R18, R19, R2, R3, R4, R7, R8, R9: device rcl:R-US_R0402 -> rcl:R-US_R0201
- R20, R21: value (none) -> 47K; device rcl:R-US_R0402 -> rcl:R-US_R0201
- X1: value USBPCB -> CRYSTAL-ABRACON-ABM11; device Pygmy:USBPCB -> Pygmy:CRYSTAL-ABRACON-ABM11
Connections:
- net EXT0: now also U2.PA3; no longer U2.PA0-WKUP
- net EXT3: now also U2.PA0-WKUP; no longer U2.PA3
- net GND: now also JP1.GND, X1G$2.GND@1, X1G$2.GND@2; no longer X1.GND
- net N$1: now also JP1.D+; no longer X1.D+
- net N$2: now also JP1.D-; no longer X1.D-
- net N$9: now also JP1.VBUS; no longer X1.VBUS
- net OSC32_IN: now also X2.2; no longer Q2.XOUT
- net OSC32_OUT: now also X2.1; no longer Q2.XIN
- net OSC_IN: now also X1G$1.2; no longer Q1.2
- net OSC_OUT: now also X1G$1.1; no longer Q1.1
